Commit message: Created a dummy_robot simulations in gazebo works

File: urdf/depthai_descr.urdf.xacro (robot description, xacro)
@@ -4,10 +4,10 @@
     <xacro:arg name="camera_model"  default="OAK-D" />
     <xacro:arg name="base_frame"    default="oak-d_frame" />
-    <xacro:arg name="parent_frame"  default="button_power" />
-    <xacro:arg name="cam_pos_x"     default="0.0" />
+    <xacro:arg name="parent_frame"  default="base_link" />
+    <xacro:arg name="cam_pos_x"     default="0.2" />
     <xacro:arg name="cam_pos_y"     default="0.0" />
-    <xacro:arg name="cam_pos_z"     default="0.0" />
+    <xacro:arg name="cam_pos_z"     default="0.2" />
     <xacro:arg name="cam_roll"      default="0.0" />
-    <xacro:arg name="cam_pitch"     default="1.57" />
+    <xacro:arg name="cam_pitch"     default="0.0" />
     <xacro:arg name="cam_yaw"       default="0.0" />
     <xacro:include filename="$(find simulation)/urdf/include/depthai_macro.urdf.xacro"/>

File: urdf/include/depthai_macro.urdf.xacro (robot description, xacro)
@@ -23,14 +23,9 @@
     <link name="${base_frame}">
         <collision>
-            <origin xyz="0 0 -1" rpy="0 0 0"/>
+            <origin xyz="0 0 0" rpy="0 0 0"/>
             <geometry>
                <box size="0.1 0.05 0.05"/>
             </geometry>
         </collision>
-                <inertial>
-            <mass value="1" />
-            <origin rpy="0 0 0" xyz="0 0 0"/>
-            <inertia ixx="0" ixy="0" ixz="0" iyy="0" iyz="0" izz="0" />
-        </inertial>
     </link>
     <joint name="${camera_name}_center_joint" type="fixed">

File: urdf/robot.urdf.xacro (robot description, xacro)
@@ -2,5 +2,6 @@
 <robot name="turtlebot4" xmlns:xacro="http://ros.org/wiki/xacro">
   <!-- Base create3 model -->
-    <xacro:include filename="$(find simulation)/urdf/irobot_create_description/urdf/create3.urdf.xacro" />
+    <xacro:include filename="$(find simulation)/urdf/dummy_robot/robot_core.xacro" />
+    <xacro:include filename="$(find simulation)/urdf/dummy_robot/gazebo_control.xacro" />
     <xacro:include filename="$(find simulation)/urdf/depthai_descr.urdf.xacro" />
 </robot>
