Commit message: bug OLD_DATA fixed and added base_fotprint to urdf

File: urdf/irobot_create_description/urdf/create3.urdf.xacro (robot description, xacro)
@@ -70,4 +70,17 @@
     </gazebo>
   </xacro:if>
+  <!-- Footprint -->
+  <link name="base_footprint"/>
+  <joint name="base_joint" type="fixed">
+    <parent link="base_link"/>
+    <child link="base_footprint"/>
+    <origin xyz="0.0 0.0 0.0" rpy="0 0 0"/>
+  </joint>
+  <link name="map"/>
+  <joint name="map_joint" type="fixed">
+    <parent link="base_link"/>
+    <child link="map"/>
+    <origin xyz="0.0 0.0 0.0" rpy="0 0 0"/>
+  </joint>
   <!-- Bumper -->
   <xacro:bumper

File: urdf/oak-D/include/depthai_macro.urdf.xacro (robot description, xacro)
@@ -73,6 +73,5 @@
         <child link="${camera_name}_rgb_camera_optical_frame"/>
     </joint>
-    <gazebo reference="${camera_name}_rgb_camera_frame">
-        <material>Gazebo/Red</material>
+     <gazebo reference="${camera_name}_rgb_camera_frame">
         <sensor name="camera" type="depth">
             <pose> 0 0 0 0 0 0 </pose>

File: urdf/turtlebot4_description/urdf/sensors/rplidar.urdf.xacro (robot description, xacro)
@@ -29,13 +29,32 @@
     <xacro:inertial_cuboid mass="0.17" x="${length_x}" y="${length_y}" z="${length_z}"/>
   </link>
-  <gazebo reference="${name}_link">
-    <xacro:ray_sensor sensor_name="${name}" gazebo="${gazebo}"
-                  update_rate="62.0" visualize="1"
-                  h_samples="640" h_res="1.0" h_min_angle="${-pi}" h_max_angle="${pi}"
-                  r_min="0.164" r_max="12.0" r_res="0.01">
-                  <plugin name="dummy" filename="dummyfile"></plugin>
-    </xacro:ray_sensor>
-    <xacro:material_darkgray/>
-  </gazebo>
+    <gazebo reference="${name}_link">
+        <material>Gazebo/Black</material>
+        <sensor name="laser" type="ray">
+            <visualize>true</visualize>
+            <update_rate>10</update_rate>
+            <ray>
+                <scan>
+                    <horizontal>
+                        <samples>180</samples>
+                        <resolution>2</resolution>
+                        <min_angle>-3.14</min_angle>
+                        <max_angle>3.14</max_angle>
+                    </horizontal>
+                </scan>
+                <range>
+                    <min>0.2</min>
+                    <max>10</max>
+                </range>
+            </ray>
+            <plugin name="laser_controller" filename="libgazebo_ros_ray_sensor.so">
+              <ros>
+                  <argument>~/out:=scan</argument>
+              </ros>
+                <output_type>sensor_msgs/LaserScan</output_type>
+            <frameName>${name}_link</frameName>
+            </plugin>
+        </sensor>
+    </gazebo>
   <gazebo reference="${name}_joint">
     <preserveFixedJoint>true</preserveFixedJoint>
